Commit message: Added the rear lidar to URDF and changed the IMU and front lidar positions. Enlarged car collision geometry. #11

File: gigatron_hardware/urdf/gigatron_testing.urdf.xacro (robot description, xacro)
@@ -3,13 +3,8 @@
     xmlns:xacro="http://www.ros.org/wiki/xacro"
     name="gigatron">
-    <!-- Note: Base Link is the center of the robot, right under the batteries. -->
     <!-- Physical Constant Macros -->
     <xacro:property name="M_PI" value="3.1415926535897931" />
     <!-- Dimension Macros -->
-    <xacro:property name="car_length" value="1.257" />
-    <!--28.5" front to back wheel axes
-        Front bumper is 25.5" (0.6477m) front from base,
-        Rear bumper is 24" (0.6096m) from base. 1.5" offset.-->
-    <xacro:property name="wheelbase_length" value="0.7239" />
+    <xacro:property name="car_length" value="0.7239" /> <!-- 28.5" front to back wheel axes -->
     <xacro:property name="wheelbase_width" value="0.5842" /> <!-- 24" -->
     <xacro:property name="car_height" value="0.2794" /> <!-- 11"? -->
@@ -19,15 +14,10 @@
     <xacro:property name="imu_x" value="0" />
     <xacro:property name="imu_y" value="0" />
-    <xacro:property name="imu_z" value="-.5" /> <!-- TODO: Update this value. This one is temporary. -->
+    <xacro:property name="imu_z" value="0.22862" />
     <!-- LIDAR placement relative to base_link -->
-    <xacro:property name="lidar_x" value=".5588" />
-    <xacro:property name="lidar_y" value="0" />
-    <xacro:property name="lidar_z" value="0.2286" />
+    <xacro:property name="lidar_x" value="-0.0254" />
+    <xacro:property name="lidar_y" value="0.1524" />
+    <xacro:property name="lidar_z" value="0.27942" />
     <xacro:property name="lidar_yaw" value="${M_PI}" />
-    <!-- Rear LIDAR placement relative to base_link -->
-    <xacro:property name="back_lidar_x" value="-0.5334" />
-    <xacro:property name="back_lidar_y" value="0" />
-    <xacro:property name="back_lidar_z" value="0.3048" />
-    <xacro:property name="back_lidar_yaw" value="0" />
     <!-- Physical Material Macros -->
     <material name="Grey">
@@ -58,5 +48,5 @@
         </visual>
         <collision>
-            <origin xyz=".031 0 0" rpy="0 0 0" />
+            <origin xyz="0 0 0" rpy="0 0 0" />
             <geometry>
                 <box size="${car_length} ${wheelbase_width} ${car_height}" />
@@ -70,5 +60,5 @@
         <parent link="base_link" />
         <child link="front_left_wheel_link" />
-        <origin xyz="${wheelbase_length/2} -${wheelbase_width/2} -${wheel_radius}" rpy="0 0 0" /> <!-- ? -->
+        <origin xyz="${car_length/2} -${wheelbase_width/2} -${wheel_radius}" rpy="0 0 0" /> <!-- ? -->
     </joint>
     <link name="front_left_wheel_link">
@@ -98,5 +88,5 @@
         <parent link="base_link" />
         <child link="front_right_wheel_link" />
-        <origin xyz="${wheelbase_length/2} ${wheelbase_width/2} -${wheel_radius}" rpy="0 0 0" /> <!-- ? -->
+        <origin xyz="${car_length/2} ${wheelbase_width/2} -${wheel_radius}" rpy="0 0 0" /> <!-- ? -->
     </joint>
     <link name="front_right_wheel_link">
@@ -125,5 +115,5 @@
         <parent link="base_link" />
         <child link="back_left_wheel_link" />
-        <origin xyz="-${wheelbase_length/2} -${wheelbase_width/2} -${wheel_radius}" rpy="0 0 0" /> <!-- ? -->
+        <origin xyz="-${car_length/2} -${wheelbase_width/2} -${wheel_radius}" rpy="0 0 0" /> <!-- ? -->
     </joint>
     <link name="back_left_wheel_link">
@@ -152,5 +142,5 @@
         <parent link="base_link" />
         <child link="back_right_wheel_link" />
-        <origin xyz="-${wheelbase_length/2} ${wheelbase_width/2} -${wheel_radius}" rpy="0 0 0" /> <!-- ? -->
+        <origin xyz="-${car_length/2} ${wheelbase_width/2} -${wheel_radius}" rpy="0 0 0" /> <!-- ? -->
     </joint>
     <link name="back_right_wheel_link">
@@ -200,30 +190,4 @@
         </collision>
     </link>
-    <!-- BACK LIDAR -->
-    <joint name="back_laser_base_mount_joint" type="fixed">
-        <origin xyz="${back_lidar_x} ${back_lidar_y} ${back_lidar_z}" rpy="0 0 ${back_lidar_yaw}" />
-        <parent link="base_link"/>
-        <child link="back_laser_link"/>
-    </joint>
-    <link name="back_laser_link" type="fixed">
-        <inertial>
-            <mass value="0.1"/>
-            <origin xyz="0 0 0.0"/>
-            <inertia ixx="0.1" ixy="0" ixz="0" iyy="0.1" iyz="0" izz="0.1"/>
-        </inertial>
-        <visual>
-            <origin rpy="0 0 0" xyz="0 0 0.02"/>
-            <geometry>
-                <cylinder radius="0.04" length="0.03175"/>
-            </geometry>
-            <material name="DarkGrey"/>
-        </visual>
-        <collision>
-            <origin rpy="0 0 0" xyz="0 0 0.025"/>
-            <geometry>
-                <box size="0.05 0.05 0.05"/>
-            </geometry>
-        </collision>
-    </link>
     <!-- IMU -->
     <joint name="imu_mount_joint" type="fixed">
@@ -245,4 +209,10 @@
             <material name="Blue"/>
         </visual>
+        <collision>
+            <origin xyz="0 0 0" rpy="0 0 0" />
+            <geometry>
+                <box size="${car_length} ${wheelbase_width} ${car_height}" />
+            </geometry>
+        </collision>
     </link>
 </robot>
