Commit message: Fixed all of the laser problems maybe

File: gigatron_hardware/urdf/kilotron.urdf.xacro (robot description, xacro)
@@ -121,6 +121,6 @@
     </gazebo>
 	<!-- the back left wheel -->
-    <joint name="back_left_wheel_joint" type="continuous" >
-        <axis xyz="0 1 0" />
+    <joint name="back_left_wheel_joint" type="fixed" >
+        <!-- <axis xyz="0 1 0" /> -->
         <parent link="base_link" />
         <child link="back_left_wheel_link" />
@@ -151,6 +151,6 @@
     </gazebo>
 	<!-- the back right wheel -->
-    <joint name="back_right_wheel_joint" type="continuous" >
-        <axis xyz="0 1 0" />
+    <joint name="back_right_wheel_joint" type="fixed" >
+        <!-- <axis xyz="0 1 0" /> -->
         <parent link="base_link" />
         <child link="back_right_wheel_link" />
@@ -213,5 +213,5 @@
 z: 0.1143   # 4.5" up from wheel axis -->
         <joint name="laser_base_mount_joint" type="fixed">
-            <origin xyz="0.1016 0 0.05715" rpy="0 0 0" />
+            <origin xyz="0.1016 0 0.05715" rpy="0 0 ${M_PI}" />
             <parent link="base_link"/>
             <child link="laser_link"/>

Commit message: Added ZED to Kilotron URDF #22

File: gigatron_hardware/urdf/kilotron.urdf.xacro (robot description, xacro)
@@ -20,4 +20,8 @@
     <xacro:property name="lidar_z" value="0.05715" />
     <xacro:property name="lidar_yaw" value="${M_PI}" />
+    <!-- ZED placement relative to base_link -->
+    <xacro:property name="zed_x" value="0.1778" />
+    <xacro:property name="zed_y" value="0" />
+    <xacro:property name="zed_z" value="0" /> <!-- or 0.0381 up from wheel axis? -->
     <!-- Physical Material Macros -->
     <material name="Grey">
@@ -216,3 +220,39 @@
         </collision>
     </link>
+    <!-- ZED -->
+    <joint name="zed_joint" type="fixed">
+        <origin xyz="${zed_x} ${zed_y} ${zed_z}" rpy="0 0 0" />
+        <parent link="base_link"/>
+        <child link="zed_link"/>
+    </joint>
+    <link name="zed_link" type="fixed">
+        <inertial>
+            <mass value="0.2" />
+            <origin xyz="0 0 0" />
+            <inertia  ixx="0.2" ixy="0.0"  ixz="0.0"  iyy="0.2"  iyz="0.0"  izz="0.2" />
+        </inertial>
+        <visual>
+            <origin xyz="0 0 0" rpy="0 0 0" />
+            <geometry>
+                <box size="0.0381 0.1717 0.0317" /> <!-- IMU dimensions -->
+            </geometry>
+            <material name="Blue"/>
+        </visual>
+        <collision>
+            <origin xyz="0 0 0" rpy="0 0 0" />
+            <geometry>
+                <box size="${car_length} ${wheelbase_width} ${car_height}" />
+            </geometry>
+        </collision>
+    </link>
+    <!-- optical rotation -->
+    <joint name="zed_optical_joint" type="fixed">
+        <origin xyz="0 0 0" rpy="${-M_PI/2} 0 ${-M_PI/2}" />
+        <parent link="zed_link"/>
+        <child link="zed_optical_frame"/>
+    </joint>
+    <link name="zed_optical_frame" type="fixed">
+        <inertia ixx="0.0001" ixy="0.0" ixz="0.0" iyy="0.0001" iyz="0.0" izz="0.0001" />
+        </inertial>
+    </link>
 </robot>

Commit message: Fixed kilotron launch file and URDF

File: gigatron_hardware/urdf/kilotron.urdf.xacro (robot description, xacro)
@@ -253,5 +253,8 @@
     </joint>
     <link name="zed_optical_frame" type="fixed">
-        <inertia ixx="0.0001" ixy="0.0" ixz="0.0" iyy="0.0001" iyz="0.0" izz="0.0001" />
+        <inertial>
+            <mass value="0.0001" />
+            <origin xyz="0 0 0" />
+            <inertia ixx="0.0001" ixy="0.0" ixz="0.0" iyy="0.0001" iyz="0.0" izz="0.0001" />
         </inertial>
     </link>

Commit message: Added ZED left and right optical frames to Kilotron URDF #22

File: gigatron_hardware/urdf/kilotron.urdf.xacro (robot description, xacro)
@@ -23,5 +23,6 @@
     <xacro:property name="zed_x" value="0.1778" />
     <xacro:property name="zed_y" value="0" />
-    <xacro:property name="zed_z" value="0" /> <!-- or 0.0381 up from wheel axis? -->
+    <xacro:property name="zed_z" value="0" />
+    <xacro:property name="zed_cam_separation" value="0.12065" />
     <!-- Physical Material Macros -->
     <material name="Grey">
@@ -255,5 +256,5 @@
     <!-- optical rotation -->
     <joint name="zed_optical_joint" type="fixed">
-        <origin xyz="0 0 0" rpy="${-M_PI/2} 0 ${-M_PI/2}" />
+        <origin xyz="${0.0381/2} 0 0" rpy="${-M_PI/2} 0 ${-M_PI/2}" />
         <parent link="zed_link"/>
         <child link="zed_optical_frame"/>
@@ -266,3 +267,53 @@
         </inertial>
     </link>
+    <!-- left camera -->
+    <joint name="zed_left_camera_joint" type="fixed">
+        <origin xyz="${0.0381/2} ${zed_cam_separation/2} 0" rpy="0 0 0" />
+        <parent link="zed_link"/>
+        <child link="left_camera_link"/>
+    </joint>
+    <link name="left_camera_link" type="fixed">
+        <inertial>
+            <mass value="0.0001" />
+            <origin xyz="0 0 0" />
+            <inertia ixx="0.0001" ixy="0.0" ixz="0.0" iyy="0.0001" iyz="0.0" izz="0.0001" />
+        </inertial>
+    </link>
+    <joint name="left_optical_joint" type="fixed">
+        <origin xyz="0 0 0" rpy="${-M_PI/2} 0 ${-M_PI/2}" />
+        <parent link="left_camera_link"/>
+        <child link="left_optical_frame"/>
+    </joint>
+    <link name="left_optical_frame" type="fixed">
+        <inertial>
+            <mass value="0.0001" />
+            <origin xyz="0 0 0" />
+            <inertia ixx="0.0001" ixy="0.0" ixz="0.0" iyy="0.0001" iyz="0.0" izz="0.0001" />
+        </inertial>
+    </link>
+    <!-- right camera -->
+    <joint name="zed_right_camera_joint" type="fixed">
+        <origin xyz="${0.0381/2} -${zed_cam_separation/2} 0" rpy="0 0 0" />
+        <parent link="zed_link"/>
+        <child link="right_camera_link"/>
+    </joint>
+    <link name="right_camera_link" type="fixed">
+        <inertial>
+            <mass value="0.0001" />
+            <origin xyz="0 0 0" />
+            <inertia ixx="0.0001" ixy="0.0" ixz="0.0" iyy="0.0001" iyz="0.0" izz="0.0001" />
+        </inertial>
+    </link>
+    <joint name="right_optical_joint" type="fixed">
+        <origin xyz="0 0 0" rpy="${-M_PI/2} 0 ${-M_PI/2}" />
+        <parent link="right_camera_link"/>
+        <child link="right_optical_frame"/>
+    </joint>
+    <link name="right_optical_frame" type="fixed">
+        <inertial>
+            <mass value="0.0001" />
+            <origin xyz="0 0 0" />
+            <inertia ixx="0.0001" ixy="0.0" ixz="0.0" iyy="0.0001" iyz="0.0" izz="0.0001" />
+        </inertial>
+    </link>
 </robot>

Commit message: Updated kilotron launch and URDF for XV LIDAR

File: gigatron_hardware/urdf/kilotron.urdf.xacro (robot description, xacro)
@@ -21,5 +21,5 @@
     <xacro:property name="lidar_y" value="0" />
     <xacro:property name="lidar_z" value="0.05715" />
-    <xacro:property name="lidar_yaw" value="${M_PI}" />
+    <xacro:property name="lidar_yaw" value="0" />
     <!-- ZED placement relative to base_link -->
     <xacro:property name="zed_x" value="0.1778" />
@@ -166,6 +166,6 @@
     </link>
     <!-- RPLIDAR -->
-    <xacro:rplidar_v0
-        name="rplidar"
+    <xacro:xvlidar_v0
+        name="xvlidar"
         parent="base_link">
         <origin
