Commit message: Added urdf.xacro template for Gigatron

File: gigatron_hardware/urdf/gigatron.urdf.xacro (robot description, xacro)
@@ -1,9 +1,20 @@
 <?xml version="1.0"?>
 <robot
+    xmlns:gazebo="http://playerstage.sourceforge.net/gazebo/xmlschema/#gz"
+    xmlns:model="http://playerstage.sourceforge.net/gazebo/xmlschema/#model"
+    xmlns:sensor="http://playerstage.sourceforge.net/gazebo/xmlschema/#sensor"
+    xmlns:body="http://playerstage.sourceforge.net/gazebo/xmlschema/#body"
+    xmlns:geom="http://playerstage.sourceforge.net/gazebo/xmlschema/#geom"
+    xmlns:joint="http://playerstage.sourceforge.net/gazebo/xmlschema/#joint"
+    xmlns:controller="http://playerstage.sourceforge.net/gazebo/xmlschema/#controller"
+    xmlns:interface="http://playerstage.sourceforge.net/gazebo/xmlschema/#interface"
+    xmlns:rendering="http://playerstage.sourceforge.net/gazebo/xmlschema/#rendering"
+    xmlns:physics="http://playerstage.sourceforge.net/gazebo/xmlschema/#physics"
     xmlns:xacro="http://www.ros.org/wiki/xacro"
-    name="kilotron">
+    name="gigatron">
     <!-- Physical Constant Macros -->
     <xacro:property name="M_PI" value="3.1415926535897931" />
     <!-- Dimension Macros -->
+    <!-- TODO: update with values for Gigatron -->
     <xacro:property name="car_length" value="0.254" /> <!-- 10" -->
     <xacro:property name="wheelbase_width" value="0.1778" />
@@ -16,11 +27,11 @@
     </material>
     <material name="Blue">
-        <color rgba="0 0 1.0 0.5"/>
+    	<color rgba="0 0 1.0 0.5"/>
     </material>
     <material name="Black">
-        <color rgba="0 0 0 1.0"/>
+    	<color rgba="0 0 0 1.0"/>
     </material>
     <material name="Aqua">
-        <color rgba="0 255 255 1.0"/>
+    	<color rgba="0 255 255 1.0"/>
     </material>
     <!-- Main body -->
@@ -45,4 +56,7 @@
         </collision>
     </link>
+    <gazebo reference="base_link">
+        <material>Gazebo/Grey</material>
+    </gazebo>
     <!-- the front left wheel -->
     <joint name="front_left_wheel_joint" type="revolute" >
@@ -73,4 +87,7 @@
         </collision>
     </link>
+    <gazebo reference="front_left_wheel_link">
+        <material>Gazebo/Black</material>
+    </gazebo>
     <!-- the front right wheel -->
     <joint name="front_right_wheel_joint" type="revolute" >
@@ -101,5 +118,8 @@
         </collision>
     </link>
-    <!-- the back left wheel -->
+    <gazebo reference="front_right_wheel_link">
+        <material>Gazebo/Black</material>
+    </gazebo>
+	<!-- the back left wheel -->
     <joint name="back_left_wheel_joint" type="fixed" >
         <!-- <axis xyz="0 1 0" /> -->
@@ -128,5 +148,8 @@
         </collision>
     </link>
-    <!-- the back right wheel -->
+    <gazebo reference="back_left_wheel_link">
+        <material>Gazebo/Black</material>
+    </gazebo>
+	<!-- the back right wheel -->
     <joint name="back_right_wheel_joint" type="fixed" >
         <!-- <axis xyz="0 1 0" /> -->
@@ -155,28 +178,88 @@
         </collision>
     </link>
-    <!-- LIDAR -->
-    <joint name="laser_base_mount_joint" type="fixed">
-        <origin xyz="0.1016 0 0.05715" rpy="0 0 ${M_PI}" />
-        <parent link="base_link"/>
-        <child link="laser_link"/>
-    </joint>
-    <link name="laser_link" type="fixed">
-        <inertial>
-            <mass value="0.1"/>
-            <origin xyz="0 0 0.0"/>
-            <inertia ixx="0.1" ixy="0" ixz="0" iyy="0.1" iyz="0" izz="0.1"/>
-        </inertial>
-        <visual>
-            <origin rpy="0 0 0" xyz="0 0 0.02"/>
-            <geometry>
-                <cylinder radius="0.04" length="0.03175"/>
-            </geometry>
-        </visual>
-        <collision>
-            <origin rpy="0 0 0" xyz="0 0 0.025"/>
-            <geometry>
-                <box size="0.05 0.05 0.05"/>
-            </geometry>
-        </collision>
-    </link>
-</robot>
+    <gazebo reference="back_right_wheel_link">
+        <material>Gazebo/Black</material>
+    </gazebo>
+    <!-- Ackermann plugin -->
+    <gazebo>
+      <controller:ackermann_plugin name="ackermann_controller"
+			           plugin="libackermann_plugin.so">
+	<alwaysOn>true</alwaysOn>
+	<update>100</update>
+	<updateRate>100.0</updateRate>
+	<leftJoint>back_left_wheel_joint</leftJoint>
+	<rightJoint>back_right_wheel_joint</rightJoint>
+	<steerJoint>steer_joint</steerJoint>
+	<wheelSeparationWidth>0.16</wheelSeparationWidth>
+	<wheelSeparationLength>0.32</wheelSeparationLength>
+	<wheelDiameter>0.041</wheelDiameter>
+	<driveTorque>5</driveTorque>
+	<steerTorque>5</steerTorque>
+	<interface:position name="position_iface_0" />
+	<robotNamespace>/</robotNamespace>
+	<topicName>pilot/drive</topicName>
+      </controller:ackermann_plugin>
+     <canonicalBody>base_footprint</canonicalBody>
+    <!-- this publishes empty joint_states due to no transmission, but
+    triggering robot_state_publisher to publish tf between fixed joints in erratic,
+    (e.g. base_laser_link for the base_scan frame) -->
+    <controller:gazebo_ros_controller_manager name="gazebo_ros_controller_manager" plugin="libgazebo_ros_controller_manager.so">
+      <alwaysOn>true</alwaysOn>
+      <updateRate>100.0</updateRate>
+      <interface:audio name="gazebo_ros_controller_manager_dummy_iface" />
+    </controller:gazebo_ros_controller_manager>
+    </gazebo>
+<!-- x: 0.1016   # 4" forward from center of car
+y: 0        # center of car
+z: 0.1143   # 4.5" up from wheel axis -->
+        <joint name="laser_base_mount_joint" type="fixed">
+            <origin xyz="0.1016 0 0.05715" rpy="0 0 ${M_PI}" />
+            <parent link="base_link"/>
+            <child link="laser_link"/>
+        </joint>
+        <link name="laser_link" type="fixed">
+            <inertial>
+                <mass value="0.1"/>
+                <origin xyz="0 0 0.0"/>
+                <inertia ixx="0.1" ixy="0" ixz="0" iyy="0.1" iyz="0" izz="0.1"/>
+            </inertial>
+            <visual>
+                <origin rpy="0 0 0" xyz="0 0 0.02"/>
+                <geometry>
+                    <cylinder radius="0.04" length="0.03175"/>
+                </geometry>
+            </visual>
+            <collision>
+                <origin rpy="0 0 0" xyz="0 0 0.025"/>
+                <geometry>
+                    <box size="0.05 0.05 0.05"/>
+                </geometry>
+            </collision>
+        </link>
+        <gazebo reference="laser_link">
+            <sensor:ray name="laser">
+                <rayCount>683</rayCount>
+                <rangeCount>683</rangeCount>
+                <laserCount>1</laserCount>
+                <origin>0.0 0.0 0.0</origin>
+                <displayRays>false</displayRays>
+                <minAngle>-135</minAngle>
+                <maxAngle> 135</maxAngle>
+                <minRange>0.06</minRange>
+                <maxRange>4.0</maxRange>
+                <resRange>0.001</resRange>
+                <updateRate>10.0</updateRate>
+                <controller:gazebo_ros_laser name="gazebo_ros_base_scan_link_controller" plugin="libgazebo_ros_laser.so">
+                    <gaussianNoise>0.005</gaussianNoise>
+                    <alwaysOn>true</alwaysOn>
+                    <updateRate>10.0</updateRate>
+                    <topicName>scan</topicName>
+                    <frameName>laser_link</frameName>
+                    <interface:laser name="gazebo_ros_base_scan_link_iface"/>
+                </controller:gazebo_ros_laser>
+            </sensor:ray>
+        </gazebo>
+        <gazebo reference="laser_link">
+            <material>Gazebo/Black</material>
+        </gazebo>
+	</robot>

Commit message: Simplifying hardware launch files

File: gigatron_hardware/urdf/gigatron.urdf.xacro (robot description, xacro)
@@ -1,14 +1,4 @@
 <?xml version="1.0"?>
 <robot
-    xmlns:gazebo="http://playerstage.sourceforge.net/gazebo/xmlschema/#gz"
-    xmlns:model="http://playerstage.sourceforge.net/gazebo/xmlschema/#model"
-    xmlns:sensor="http://playerstage.sourceforge.net/gazebo/xmlschema/#sensor"
-    xmlns:body="http://playerstage.sourceforge.net/gazebo/xmlschema/#body"
-    xmlns:geom="http://playerstage.sourceforge.net/gazebo/xmlschema/#geom"
-    xmlns:joint="http://playerstage.sourceforge.net/gazebo/xmlschema/#joint"
-    xmlns:controller="http://playerstage.sourceforge.net/gazebo/xmlschema/#controller"
-    xmlns:interface="http://playerstage.sourceforge.net/gazebo/xmlschema/#interface"
-    xmlns:rendering="http://playerstage.sourceforge.net/gazebo/xmlschema/#rendering"
-    xmlns:physics="http://playerstage.sourceforge.net/gazebo/xmlschema/#physics"
     xmlns:xacro="http://www.ros.org/wiki/xacro"
     name="gigatron">
@@ -16,5 +6,5 @@
     <xacro:property name="M_PI" value="3.1415926535897931" />
     <!-- Dimension Macros -->
-    <!-- TODO: update with values for Gigatron -->
+    <!-- TODO: replace with Gigatron values -->
     <xacro:property name="car_length" value="0.254" /> <!-- 10" -->
     <xacro:property name="wheelbase_width" value="0.1778" />
@@ -27,11 +17,11 @@
     </material>
     <material name="Blue">
-    	<color rgba="0 0 1.0 0.5"/>
+        <color rgba="0 0 1.0 0.5"/>
     </material>
     <material name="Black">
-    	<color rgba="0 0 0 1.0"/>
+        <color rgba="0 0 0 1.0"/>
     </material>
     <material name="Aqua">
-    	<color rgba="0 255 255 1.0"/>
+        <color rgba="0 255 255 1.0"/>
     </material>
     <!-- Main body -->
@@ -56,7 +46,4 @@
         </collision>
     </link>
-    <gazebo reference="base_link">
-        <material>Gazebo/Grey</material>
-    </gazebo>
     <!-- the front left wheel -->
     <joint name="front_left_wheel_joint" type="revolute" >
@@ -87,7 +74,4 @@
         </collision>
     </link>
-    <gazebo reference="front_left_wheel_link">
-        <material>Gazebo/Black</material>
-    </gazebo>
     <!-- the front right wheel -->
     <joint name="front_right_wheel_joint" type="revolute" >
@@ -118,8 +102,5 @@
         </collision>
     </link>
-    <gazebo reference="front_right_wheel_link">
-        <material>Gazebo/Black</material>
-    </gazebo>
-	<!-- the back left wheel -->
+    <!-- the back left wheel -->
     <joint name="back_left_wheel_joint" type="fixed" >
         <!-- <axis xyz="0 1 0" /> -->
@@ -148,8 +129,5 @@
         </collision>
     </link>
-    <gazebo reference="back_left_wheel_link">
-        <material>Gazebo/Black</material>
-    </gazebo>
-	<!-- the back right wheel -->
+    <!-- the back right wheel -->
     <joint name="back_right_wheel_joint" type="fixed" >
         <!-- <axis xyz="0 1 0" /> -->
@@ -178,88 +156,28 @@
         </collision>
     </link>
-    <gazebo reference="back_right_wheel_link">
-        <material>Gazebo/Black</material>
-    </gazebo>
-    <!-- Ackermann plugin -->
-    <gazebo>
-      <controller:ackermann_plugin name="ackermann_controller"
-			           plugin="libackermann_plugin.so">
-	<alwaysOn>true</alwaysOn>
-	<update>100</update>
-	<updateRate>100.0</updateRate>
-	<leftJoint>back_left_wheel_joint</leftJoint>
-	<rightJoint>back_right_wheel_joint</rightJoint>
-	<steerJoint>steer_joint</steerJoint>
-	<wheelSeparationWidth>0.16</wheelSeparationWidth>
-	<wheelSeparationLength>0.32</wheelSeparationLength>
-	<wheelDiameter>0.041</wheelDiameter>
-	<driveTorque>5</driveTorque>
-	<steerTorque>5</steerTorque>
-	<interface:position name="position_iface_0" />
-	<robotNamespace>/</robotNamespace>
-	<topicName>pilot/drive</topicName>
-      </controller:ackermann_plugin>
-     <canonicalBody>base_footprint</canonicalBody>
-    <!-- this publishes empty joint_states due to no transmission, but
-    triggering robot_state_publisher to publish tf between fixed joints in erratic,
-    (e.g. base_laser_link for the base_scan frame) -->
-    <controller:gazebo_ros_controller_manager name="gazebo_ros_controller_manager" plugin="libgazebo_ros_controller_manager.so">
-      <alwaysOn>true</alwaysOn>
-      <updateRate>100.0</updateRate>
-      <interface:audio name="gazebo_ros_controller_manager_dummy_iface" />
-    </controller:gazebo_ros_controller_manager>
-    </gazebo>
-<!-- x: 0.1016   # 4" forward from center of car
-y: 0        # center of car
-z: 0.1143   # 4.5" up from wheel axis -->
-        <joint name="laser_base_mount_joint" type="fixed">
-            <origin xyz="0.1016 0 0.05715" rpy="0 0 ${M_PI}" />
-            <parent link="base_link"/>
-            <child link="laser_link"/>
-        </joint>
-        <link name="laser_link" type="fixed">
-            <inertial>
-                <mass value="0.1"/>
-                <origin xyz="0 0 0.0"/>
-                <inertia ixx="0.1" ixy="0" ixz="0" iyy="0.1" iyz="0" izz="0.1"/>
-            </inertial>
-            <visual>
-                <origin rpy="0 0 0" xyz="0 0 0.02"/>
-                <geometry>
-                    <cylinder radius="0.04" length="0.03175"/>
-                </geometry>
-            </visual>
-            <collision>
-                <origin rpy="0 0 0" xyz="0 0 0.025"/>
-                <geometry>
-                    <box size="0.05 0.05 0.05"/>
-                </geometry>
-            </collision>
-        </link>
-        <gazebo reference="laser_link">
-            <sensor:ray name="laser">
-                <rayCount>683</rayCount>
-                <rangeCount>683</rangeCount>
-                <laserCount>1</laserCount>
-                <origin>0.0 0.0 0.0</origin>
-                <displayRays>false</displayRays>
-                <minAngle>-135</minAngle>
-                <maxAngle> 135</maxAngle>
-                <minRange>0.06</minRange>
-                <maxRange>4.0</maxRange>
-                <resRange>0.001</resRange>
-                <updateRate>10.0</updateRate>
-                <controller:gazebo_ros_laser name="gazebo_ros_base_scan_link_controller" plugin="libgazebo_ros_laser.so">
-                    <gaussianNoise>0.005</gaussianNoise>
-                    <alwaysOn>true</alwaysOn>
-                    <updateRate>10.0</updateRate>
-                    <topicName>scan</topicName>
-                    <frameName>laser_link</frameName>
-                    <interface:laser name="gazebo_ros_base_scan_link_iface"/>
-                </controller:gazebo_ros_laser>
-            </sensor:ray>
-        </gazebo>
-        <gazebo reference="laser_link">
-            <material>Gazebo/Black</material>
-        </gazebo>
-	</robot>
+    <!-- LIDAR -->
+    <joint name="laser_base_mount_joint" type="fixed">
+        <origin xyz="0.1016 0 0.05715" rpy="0 0 ${M_PI}" />
+        <parent link="base_link"/>
+        <child link="laser_link"/>
+    </joint>
+    <link name="laser_link" type="fixed">
+        <inertial>
+            <mass value="0.1"/>
+            <origin xyz="0 0 0.0"/>
+            <inertia ixx="0.1" ixy="0" ixz="0" iyy="0.1" iyz="0" izz="0.1"/>
+        </inertial>
+        <visual>
+            <origin rpy="0 0 0" xyz="0 0 0.02"/>
+            <geometry>
+                <cylinder radius="0.04" length="0.03175"/>
+            </geometry>
+        </visual>
+        <collision>
+            <origin rpy="0 0 0" xyz="0 0 0.025"/>
+            <geometry>
+                <box size="0.05 0.05 0.05"/>
+            </geometry>
+        </collision>
+    </link>
+</robot>

Commit message: Updated URDF for both cars

File: gigatron_hardware/urdf/gigatron.urdf.xacro (robot description, xacro)
@@ -6,22 +6,30 @@
     <xacro:property name="M_PI" value="3.1415926535897931" />
     <!-- Dimension Macros -->
-    <!-- TODO: replace with Gigatron values -->
-    <xacro:property name="car_length" value="0.254" /> <!-- 10" -->
-    <xacro:property name="wheelbase_width" value="0.1778" />
-    <xacro:property name="car_height" value="0.127" /> <!-- 5" -->
-    <xacro:property name="wheel_radius" value="0.0333" />
-    <xacro:property name="wheel_width" value="0.0254" /> <!-- 1" -->
+    <xacro:property name="car_length" value="0.7239" /> <!-- 28.5" front to back wheel axes -->
+    <xacro:property name="wheelbase_width" value="0.5842" /> <!-- 24" -->
+    <xacro:property name="car_height" value="0.2794" /> <!-- 11"? -->
+    <xacro:property name="wheel_radius" value="0.12446" /> <!-- 4.9" -->
+    <xacro:property name="wheel_width" value="0.06" /> <!-- ? -->
+    <!-- IMU placement relative to base_link -->
+    <xacro:property name="imu_x" value="0" />
+    <xacro:property name="imu_y" value="0" />
+    <xacro:property name="imu_z" value="0.22862" />
+    <!-- LIDAR placement relative to base_link -->
+    <xacro:property name="lidar_x" value="-0.0254" />
+    <xacro:property name="lidar_y" value="0.1524" />
+    <xacro:property name="lidar_z" value="0.27942" />
+    <xacro:property name="lidar_yaw" value="${M_PI}" />
     <!-- Physical Material Macros -->
     <material name="Grey">
-        <color rgba="0 0 0 0.5"/>
+        <color rgba="0 0 0 0.4"/>
     </material>
     <material name="Blue">
-        <color rgba="0 0 1.0 0.5"/>
+        <color rgba="0 0.3 0.9 0.3"/>
     </material>
     <material name="Black">
-        <color rgba="0 0 0 1.0"/>
-    </material>
-    <material name="Aqua">
-        <color rgba="0 255 255 1.0"/>
+        <color rgba="0 0 0 0.9"/>
+    </material>
+    <material name="DarkGrey">
+        <color rgba="0.5 0 0.05 0.75"/>
     </material>
     <!-- Main body -->
@@ -52,5 +60,5 @@
         <parent link="base_link" />
         <child link="front_left_wheel_link" />
-        <origin xyz="0.127 0.089 -0.0508" rpy="0 0 0" /> <!-- 5, 3.5, 2 -->
+        <origin xyz="${car_length/2} -${wheelbase_width/2} -${wheel_radius}" rpy="0 0 0" /> <!-- ? -->
     </joint>
     <link name="front_left_wheel_link">
@@ -80,5 +88,5 @@
         <parent link="base_link" />
         <child link="front_right_wheel_link" />
-        <origin xyz="0.127 -0.089 -0.0508" rpy="0 0 0" />
+        <origin xyz="${car_length/2} ${wheelbase_width/2} -${wheel_radius}" rpy="0 0 0" /> <!-- ? -->
     </joint>
     <link name="front_right_wheel_link">
@@ -107,5 +115,5 @@
         <parent link="base_link" />
         <child link="back_left_wheel_link" />
-        <origin xyz="-0.127 0.089 -0.0508" rpy="0 0 0" /> <!-- 5, 3.5, 2 -->
+        <origin xyz="-${car_length/2} -${wheelbase_width/2} -${wheel_radius}" rpy="0 0 0" /> <!-- ? -->
     </joint>
     <link name="back_left_wheel_link">
@@ -134,5 +142,5 @@
         <parent link="base_link" />
         <child link="back_right_wheel_link" />
-        <origin xyz="-0.127 -0.089 -0.0508" rpy="0 0 0" />
+        <origin xyz="-${car_length/2} ${wheelbase_width/2} -${wheel_radius}" rpy="0 0 0" /> <!-- ? -->
     </joint>
     <link name="back_right_wheel_link">
@@ -158,5 +166,5 @@
     <!-- LIDAR -->
     <joint name="laser_base_mount_joint" type="fixed">
-        <origin xyz="0.1016 0 0.05715" rpy="0 0 ${M_PI}" />
+        <origin xyz="${lidar_x} ${lidar_y} ${lidar_z}" rpy="0 0 ${lidar_yaw}" />
         <parent link="base_link"/>
         <child link="laser_link"/>
@@ -173,4 +181,5 @@
                 <cylinder radius="0.04" length="0.03175"/>
             </geometry>
+            <material name="DarkGrey"/>
         </visual>
         <collision>
@@ -181,3 +190,29 @@
         </collision>
     </link>
+    <!-- IMU -->
+    <joint name="imu_mount_joint" type="fixed">
+        <origin xyz="${imu_x} ${imu_y} ${imu_z}" rpy="0 0 0" />
+        <parent link="base_link"/>
+        <child link="imu_link"/>
+    </joint>
+    <link name="imu_link" type="fixed">
+        <inertial>
+            <mass value="0.01" />
+            <origin xyz="0 0 0" />
+            <inertia  ixx="0.2" ixy="0.0"  ixz="0.0"  iyy="0.2"  iyz="0.0"  izz="0.2" />
+        </inertial>
+        <visual>
+            <origin xyz="0 0 0" rpy="0 0 0" />
+            <geometry>
+                <box size="0.02 0.027 0.004" /> <!-- IMU dimensions -->
+            </geometry>
+            <material name="Blue"/>
+        </visual>
+        <collision>
+            <origin xyz="0 0 0" rpy="0 0 0" />
+            <geometry>
+                <box size="${car_length} ${wheelbase_width} ${car_height}" />
+            </geometry>
+        </collision>
+    </link>
 </robot>

File: gigatron_hardware/urdf/kilotron.urdf.xacro (robot description, xacro)
@@ -11,16 +11,25 @@
     <xacro:property name="wheel_radius" value="0.0333" />
     <xacro:property name="wheel_width" value="0.0254" /> <!-- 1" -->
+    <!-- IMU placement relative to base_link -->
+    <xacro:property name="imu_x" value="0" />
+    <xacro:property name="imu_y" value="0" />
+    <xacro:property name="imu_z" value="0.00637" />
+    <!-- LIDAR placement relative to base_link -->
+    <xacro:property name="lidar_x" value="0.1016" />
+    <xacro:property name="lidar_y" value="0" />
+    <xacro:property name="lidar_z" value="0.05715" />
+    <xacro:property name="lidar_yaw" value="${M_PI}" />
     <!-- Physical Material Macros -->
     <material name="Grey">
-        <color rgba="0 0 0 0.5"/>
+        <color rgba="0 0 0 0.4"/>
     </material>
     <material name="Blue">
-        <color rgba="0 0 1.0 0.5"/>
+        <color rgba="0 0.3 0.9 0.3"/>
     </material>
     <material name="Black">
-        <color rgba="0 0 0 1.0"/>
-    </material>
-    <material name="Aqua">
-        <color rgba="0 255 255 1.0"/>
+        <color rgba="0 0 0 0.9"/>
+    </material>
+    <material name="DarkGrey">
+        <color rgba="0.5 0 0.05 0.75"/>
     </material>
     <!-- Main body -->
@@ -157,5 +166,5 @@
     <!-- LIDAR -->
     <joint name="laser_base_mount_joint" type="fixed">
-        <origin xyz="0.1016 0 0.05715" rpy="0 0 ${M_PI}" />
+        <origin xyz="${lidar_x} ${lidar_y} ${lidar_z}" rpy="0 0 ${lidar_yaw}" />
         <parent link="base_link"/>
         <child link="laser_link"/>
@@ -172,4 +181,5 @@
                 <cylinder radius="0.04" length="0.03175"/>
             </geometry>
+            <material name="DarkGrey"/>
         </visual>
         <collision>
@@ -180,3 +190,29 @@
         </collision>
     </link>
+    <!-- IMU -->
+    <joint name="imu_mount_joint" type="fixed">
+        <origin xyz="${imu_x} ${imu_y} ${imu_z}" rpy="0 0 0" />
+        <parent link="base_link"/>
+        <child link="imu_link"/>
+    </joint>
+    <link name="imu_link" type="fixed">
+        <inertial>
+            <mass value="0.01" />
+            <origin xyz="0 0 0" />
+            <inertia  ixx="0.2" ixy="0.0"  ixz="0.0"  iyy="0.2"  iyz="0.0"  izz="0.2" />
+        </inertial>
+        <visual>
+            <origin xyz="0 0 0" rpy="0 0 0" />
+            <geometry>
+                <box size="0.02 0.027 0.004" /> <!-- IMU dimensions -->
+            </geometry>
+            <material name="Blue"/>
+        </visual>
+        <collision>
+            <origin xyz="0 0 0" rpy="0 0 0" />
+            <geometry>
+                <box size="${car_length} ${wheelbase_width} ${car_height}" />
+            </geometry>
+        </collision>
+    </link>
 </robot>
