Commit message: Launch and parameter file cleanup modifications

File: gigatron_hardware/urdf/gigatron.urdf.xacro (robot description, xacro)
@@ -10,5 +10,5 @@
     <xacro:property name="car_height" value="0.2794" /> <!-- 11"? -->
     <xacro:property name="wheel_radius" value="0.12446" /> <!-- 4.9" -->
-    <xacro:property name="wheel_width" value="0.06" /> <!-- ? -->
+    <xacro:property name="wheel_width" value="0.075" />
     <!-- IMU placement relative to base_link -->
     <xacro:property name="imu_x" value="0" />

Commit message: Updated gigatron.urdf.xacro with LIDAR placement changes

File: gigatron_hardware/urdf/gigatron.urdf.xacro (robot description, xacro)
@@ -24,5 +24,5 @@
     <xacro:property name="lidar_y" value="0" />
     <xacro:property name="lidar_z" value="0.2286" />
-    <xacro:property name="lidar_yaw" value="${M_PI}" />
+    <xacro:property name="lidar_yaw" value="0" />
     <!-- Rear LIDAR placement relative to base_link -->
     <xacro:property name="back_lidar_x" value="-0.5334" />

Commit message: Updated IMU mount location

File: gigatron_hardware/urdf/gigatron.urdf.xacro (robot description, xacro)
@@ -19,5 +19,5 @@
     <xacro:property name="imu_x" value="0" />
     <xacro:property name="imu_y" value="0" />
-    <xacro:property name="imu_z" value="-.5" /> <!-- TODO: Update this value. This one is temporary. -->
+    <xacro:property name="imu_z" value="-0.0254" />
     <!-- LIDAR placement relative to base_link -->
     <xacro:property name="lidar_x" value=".5588" />

Commit message: Fixed incorrect y sign for wheels in gigatron URDF and arduino_drive_controller wheel velocity visualization #17

File: gigatron_hardware/urdf/gigatron.urdf.xacro (robot description, xacro)
@@ -70,5 +70,5 @@
         <parent link="base_link" />
         <child link="front_left_wheel_link" />
-        <origin xyz="${wheelbase_length/2} -${wheelbase_width/2} -${wheel_radius}" rpy="0 0 0" /> <!-- ? -->
+        <origin xyz="${wheelbase_length/2} ${wheelbase_width/2} -${wheel_radius}" rpy="0 0 0" /> <!-- ? -->
     </joint>
     <link name="front_left_wheel_link">
@@ -98,5 +98,5 @@
         <parent link="base_link" />
         <child link="front_right_wheel_link" />
-        <origin xyz="${wheelbase_length/2} ${wheelbase_width/2} -${wheel_radius}" rpy="0 0 0" /> <!-- ? -->
+        <origin xyz="${wheelbase_length/2} -${wheelbase_width/2} -${wheel_radius}" rpy="0 0 0" /> <!-- ? -->
     </joint>
     <link name="front_right_wheel_link">
@@ -125,5 +125,5 @@
         <parent link="base_link" />
         <child link="back_left_wheel_link" />
-        <origin xyz="-${wheelbase_length/2} -${wheelbase_width/2} -${wheel_radius}" rpy="0 0 0" /> <!-- ? -->
+        <origin xyz="-${wheelbase_length/2} ${wheelbase_width/2} -${wheel_radius}" rpy="0 0 0" /> <!-- ? -->
     </joint>
     <link name="back_left_wheel_link">
@@ -152,5 +152,5 @@
         <parent link="base_link" />
         <child link="back_right_wheel_link" />
-        <origin xyz="-${wheelbase_length/2} ${wheelbase_width/2} -${wheel_radius}" rpy="0 0 0" /> <!-- ? -->
+        <origin xyz="-${wheelbase_length/2} -${wheelbase_width/2} -${wheel_radius}" rpy="0 0 0" /> <!-- ? -->
     </joint>
     <link name="back_right_wheel_link">

File: gigatron_hardware/urdf/gigatron_frame.urdf.xacro (robot description, xacro)
@@ -65,5 +65,5 @@
         <parent link="base_link" />
         <child link="front_left_wheel_link" />
-        <origin xyz="${car_length/2} -${wheelbase_width/2} -${wheel_radius}" rpy="0 0 0" /> <!-- ? -->
+        <origin xyz="${car_length/2} ${wheelbase_width/2} -${wheel_radius}" rpy="0 0 0" /> <!-- ? -->
     </joint>
     <link name="front_left_wheel_link">
@@ -93,5 +93,5 @@
         <parent link="base_link" />
         <child link="front_right_wheel_link" />
-        <origin xyz="${car_length/2} ${wheelbase_width/2} -${wheel_radius}" rpy="0 0 0" /> <!-- ? -->
+        <origin xyz="${car_length/2} -${wheelbase_width/2} -${wheel_radius}" rpy="0 0 0" /> <!-- ? -->
     </joint>
     <link name="front_right_wheel_link">
@@ -120,5 +120,5 @@
         <parent link="base_link" />
         <child link="back_left_wheel_link" />
-        <origin xyz="-${car_length/2} -${wheelbase_width/2} -${wheel_radius}" rpy="0 0 0" /> <!-- ? -->
+        <origin xyz="-${car_length/2} ${wheelbase_width/2} -${wheel_radius}" rpy="0 0 0" /> <!-- ? -->
     </joint>
     <link name="back_left_wheel_link">
@@ -147,5 +147,5 @@
         <parent link="base_link" />
         <child link="back_right_wheel_link" />
-        <origin xyz="-${car_length/2} ${wheelbase_width/2} -${wheel_radius}" rpy="0 0 0" /> <!-- ? -->
+        <origin xyz="-${car_length/2} -${wheelbase_width/2} -${wheel_radius}" rpy="0 0 0" /> <!-- ? -->
     </joint>
     <link name="back_right_wheel_link">

Commit message: Added base_footprint frame to car models

File: gigatron_hardware/urdf/gigatron.urdf.xacro (robot description, xacro)
@@ -64,4 +64,11 @@
         </collision>
     </link>
+    <!-- base_footprint (ground) to base_link -->
+    <link name="base_footprint" />
+    <joint name="base_link_footprint_joint" type="fixed" >
+        <parent link="base_footprint" />
+        <child link="base_link" />
+        <origin xyz="0 0 ${car_height/2+wheel_radius}" rpy="0 0 0" />
+    </joint>
     <!-- the front left wheel -->
     <joint name="front_left_wheel_joint" type="revolute" >

File: gigatron_hardware/urdf/gigatron_frame.urdf.xacro (robot description, xacro)
@@ -59,4 +59,11 @@
         </collision>
     </link>
+    <!-- base_footprint (ground) to base_link -->
+    <link name="base_footprint" />
+    <joint name="base_link_footprint_joint" type="fixed" >
+        <parent link="base_footprint" />
+        <child link="base_link" />
+        <origin xyz="0 0 ${car_height/2-wheel_radius}" rpy="0 0 0" />
+    </joint>
     <!-- the front left wheel -->
     <joint name="front_left_wheel_joint" type="revolute" >

File: gigatron_hardware/urdf/kilotron.urdf.xacro (robot description, xacro)
@@ -37,4 +37,11 @@
         <color rgba="0.5 0 0.05 0.75"/>
     </material>
+    <!-- base_footprint (ground) to base_link -->
+    <link name="base_footprint" />
+    <joint name="base_link_footprint_joint" type="fixed" >
+        <parent link="base_footprint" />
+        <child link="base_link" />
+        <origin xyz="0 0 ${car_height/2+0.0508-wheel_radius}" rpy="0 0 0" />
+    </joint>
     <!-- Main body -->
     <link name="base_link">

Commit message: Added ZED URDF macro #23

File: gigatron_hardware/urdf/gigatron.urdf.xacro (robot description, xacro)
@@ -3,4 +3,5 @@
     xmlns:xacro="http://www.ros.org/wiki/xacro"
     name="gigatron">
+    <xacro:include filename="$(find gigatron_hardware)/urdf/sensors/zed.urdf.xacro" />
     <!-- Note: Base Link is the center of the robot, right under the batteries. -->
     <!-- Physical Constant Macros -->
@@ -30,4 +31,8 @@
     <xacro:property name="back_lidar_z" value="0.3048" />
     <xacro:property name="back_lidar_yaw" value="0" />
+    <!-- ZED placement relative to base_link -->
+    <xacro:property name="zed_x" value="-0.0254" />
+    <xacro:property name="zed_y" value="0.0" />
+    <xacro:property name="zed_z" value="0.27942" />
     <!-- Physical Material Macros -->
     <material name="Grey">
@@ -253,3 +258,7 @@
         </visual>
     </link>
+    <!-- ZED -->
+    <xacro:zed_v0 name="zed" parent="base_link">
+        <origin xyz="${zed_x} ${zed_y} ${zed_z}" rpy="0 0 0" />
+    </xacro:zed_v0>
 </robot>

File: gigatron_hardware/urdf/kilotron.urdf.xacro (robot description, xacro)
@@ -3,6 +3,6 @@
     xmlns:xacro="http://www.ros.org/wiki/xacro"
     name="kilotron">
-    <!-- Physical Constant Macros -->
-    <xacro:property name="M_PI" value="3.1415926535897931" />
+    <xacro:include filename="$(find gigatron_hardware)/urdf/common.urdf.xacro" />
+    <xacro:include filename="$(find gigatron_hardware)/urdf/sensors/zed.urdf.xacro" />
     <!-- Dimension Macros -->
     <xacro:property name="car_length" value="0.254" /> <!-- 10" -->
@@ -25,17 +25,4 @@
     <xacro:property name="zed_z" value="0" />
     <xacro:property name="zed_cam_separation" value="0.12065" />
-    <!-- Physical Material Macros -->
-    <material name="Grey">
-        <color rgba="0 0 0 0.4"/>
-    </material>
-    <material name="Blue">
-        <color rgba="0 0.3 0.9 0.3"/>
-    </material>
-    <material name="Black">
-        <color rgba="0 0 0 0.9"/>
-    </material>
-    <material name="DarkGrey">
-        <color rgba="0.5 0 0.05 0.75"/>
-    </material>
     <!-- base_footprint (ground) to base_link -->
     <link name="base_footprint" />
@@ -229,91 +216,6 @@
     </link>
     <!-- ZED -->
-    <joint name="zed_joint" type="fixed">
+    <xacro:zed_v0 name="zed" parent="base_link">
         <origin xyz="${zed_x} ${zed_y} ${zed_z}" rpy="0 0 0" />
-        <parent link="base_link"/>
-        <child link="zed_link"/>
-    </joint>
-    <link name="zed_link" type="fixed">
-        <inertial>
-            <mass value="0.2" />
-            <origin xyz="0 0 0" />
-            <inertia  ixx="0.2" ixy="0.0"  ixz="0.0"  iyy="0.2"  iyz="0.0"  izz="0.2" />
-        </inertial>
-        <visual>
-            <origin xyz="0 0 0" rpy="0 0 0" />
-            <geometry>
-                <box size="0.0381 0.1717 0.0317" /> <!-- IMU dimensions -->
-            </geometry>
-            <material name="Blue"/>
-        </visual>
-        <collision>
-            <origin xyz="0 0 0" rpy="0 0 0" />
-            <geometry>
-                <box size="${car_length} ${wheelbase_width} ${car_height}" />
-            </geometry>
-        </collision>
-    </link>
-    <!-- optical rotation -->
-    <joint name="zed_optical_joint" type="fixed">
-        <origin xyz="${0.0381/2} 0 0" rpy="${-M_PI/2} 0 ${-M_PI/2}" />
-        <parent link="zed_link"/>
-        <child link="zed_optical_frame"/>
-    </joint>
-    <link name="zed_optical_frame" type="fixed">
-        <inertial>
-            <mass value="0.0001" />
-            <origin xyz="0 0 0" />
-            <inertia ixx="0.0001" ixy="0.0" ixz="0.0" iyy="0.0001" iyz="0.0" izz="0.0001" />
-        </inertial>
-    </link>
-    <!-- left camera -->
-    <joint name="zed_left_camera_joint" type="fixed">
-        <origin xyz="${0.0381/2} ${zed_cam_separation/2} 0" rpy="0 0 0" />
-        <parent link="zed_link"/>
-        <child link="left_camera_link"/>
-    </joint>
-    <link name="left_camera_link" type="fixed">
-        <inertial>
-            <mass value="0.0001" />
-            <origin xyz="0 0 0" />
-            <inertia ixx="0.0001" ixy="0.0" ixz="0.0" iyy="0.0001" iyz="0.0" izz="0.0001" />
-        </inertial>
-    </link>
-    <joint name="left_optical_joint" type="fixed">
-        <origin xyz="0 0 0" rpy="${-M_PI/2} 0 ${-M_PI/2}" />
-        <parent link="left_camera_link"/>
-        <child link="left_optical_frame"/>
-    </joint>
-    <link name="left_optical_frame" type="fixed">
-        <inertial>
-            <mass value="0.0001" />
-            <origin xyz="0 0 0" />
-            <inertia ixx="0.0001" ixy="0.0" ixz="0.0" iyy="0.0001" iyz="0.0" izz="0.0001" />
-        </inertial>
-    </link>
-    <!-- right camera -->
-    <joint name="zed_right_camera_joint" type="fixed">
-        <origin xyz="${0.0381/2} -${zed_cam_separation/2} 0" rpy="0 0 0" />
-        <parent link="zed_link"/>
-        <child link="right_camera_link"/>
-    </joint>
-    <link name="right_camera_link" type="fixed">
-        <inertial>
-            <mass value="0.0001" />
-            <origin xyz="0 0 0" />
-            <inertia ixx="0.0001" ixy="0.0" ixz="0.0" iyy="0.0001" iyz="0.0" izz="0.0001" />
-        </inertial>
-    </link>
-    <joint name="right_optical_joint" type="fixed">
-        <origin xyz="0 0 0" rpy="${-M_PI/2} 0 ${-M_PI/2}" />
-        <parent link="right_camera_link"/>
-        <child link="right_optical_frame"/>
-    </joint>
-    <link name="right_optical_frame" type="fixed">
-        <inertial>
-            <mass value="0.0001" />
-            <origin xyz="0 0 0" />
-            <inertia ixx="0.0001" ixy="0.0" ixz="0.0" iyy="0.0001" iyz="0.0" izz="0.0001" />
-        </inertial>
-    </link>
+    </xacro:zed_v0>
 </robot>

Commit message: Added IMU xacro macro to car .urdf.xacro files #23

File: gigatron_hardware/urdf/gigatron.urdf.xacro (robot description, xacro)
@@ -4,4 +4,7 @@
     name="gigatron">
     <xacro:include filename="$(find gigatron_hardware)/urdf/sensors/zed.urdf.xacro" />
+    <xacro:include filename="$(find gigatron_hardware)/urdf/common.urdf.xacro" />
+    <xacro:include filename="$(find gigatron_hardware)/urdf/sensors/bno055_imu.urdf.xacro" />
+    <xacro:include filename="$(find gigatron_hardware)/urdf/sensors/rplidar.urdf.xacro" />
     <!-- Note: Base Link is the center of the robot, right under the batteries. -->
     <!-- Physical Constant Macros -->
@@ -35,17 +38,4 @@
     <xacro:property name="zed_y" value="0.0" />
     <xacro:property name="zed_z" value="0.27942" />
-    <!-- Physical Material Macros -->
-    <material name="Grey">
-        <color rgba="0 0 0 0.4"/>
-    </material>
-    <material name="Blue">
-        <color rgba="0 0.3 0.9 0.3"/>
-    </material>
-    <material name="Black">
-        <color rgba="0 0 0 0.9"/>
-    </material>
-    <material name="DarkGrey">
-        <color rgba="0.5 0 0.05 0.75"/>
-    </material>
     <!-- Main body -->
     <link name="base_link">
@@ -239,23 +229,7 @@
     </link>
     <!-- IMU -->
-    <joint name="imu_mount_joint" type="fixed">
+    <xacro:bno055_imu_v0 name="imu" parent="base_link">
         <origin xyz="${imu_x} ${imu_y} ${imu_z}" rpy="0 0 0" />
-        <parent link="base_link"/>
-        <child link="imu_link"/>
-    </joint>
-    <link name="imu_link" type="fixed">
-        <inertial>
-            <mass value="0.01" />
-            <origin xyz="0 0 0" />
-            <inertia  ixx="0.2" ixy="0.0"  ixz="0.0"  iyy="0.2"  iyz="0.0"  izz="0.2" />
-        </inertial>
-        <visual>
-            <origin xyz="0 0 0" rpy="0 0 0" />
-            <geometry>
-                <box size="0.02 0.027 0.004" /> <!-- IMU dimensions -->
-            </geometry>
-            <material name="Blue"/>
-        </visual>
-    </link>
+    </xacro:bno055_imu_v0>
     <!-- ZED -->
     <xacro:zed_v0 name="zed" parent="base_link">

File: gigatron_hardware/urdf/kilotron.urdf.xacro (robot description, xacro)
@@ -5,4 +5,6 @@
     <xacro:include filename="$(find gigatron_hardware)/urdf/common.urdf.xacro" />
     <xacro:include filename="$(find gigatron_hardware)/urdf/sensors/zed.urdf.xacro" />
+    <xacro:include filename="$(find gigatron_hardware)/urdf/sensors/bno055_imu.urdf.xacro" />
+    <xacro:include filename="$(find gigatron_hardware)/urdf/sensors/rplidar.urdf.xacro" />
     <!-- Dimension Macros -->
     <xacro:property name="car_length" value="0.254" /> <!-- 10" -->
@@ -190,29 +192,7 @@
     </link>
     <!-- IMU -->
-    <joint name="imu_mount_joint" type="fixed">
+    <xacro:bno055_imu_v0 name="imu" parent="base_link">
         <origin xyz="${imu_x} ${imu_y} ${imu_z}" rpy="0 0 0" />
-        <parent link="base_link"/>
-        <child link="imu_link"/>
-    </joint>
-    <link name="imu_link" type="fixed">
-        <inertial>
-            <mass value="0.01" />
-            <origin xyz="0 0 0" />
-            <inertia  ixx="0.2" ixy="0.0"  ixz="0.0"  iyy="0.2"  iyz="0.0"  izz="0.2" />
-        </inertial>
-        <visual>
-            <origin xyz="0 0 0" rpy="0 0 0" />
-            <geometry>
-                <box size="0.02 0.027 0.004" /> <!-- IMU dimensions -->
-            </geometry>
-            <material name="Blue"/>
-        </visual>
-        <collision>
-            <origin xyz="0 0 0" rpy="0 0 0" />
-            <geometry>
-                <box size="${car_length} ${wheelbase_width} ${car_height}" />
-            </geometry>
-        </collision>
-    </link>
+    </xacro:bno055_imu_v0>
     <!-- ZED -->
     <xacro:zed_v0 name="zed" parent="base_link">

File: gigatron_hardware/urdf/sensors/bno055_imu.urdf.xacro (robot description, xacro)
@@ -2,5 +2,5 @@
 <robot xmlns:xacro="http://ros.org/wiki/xacro">
   <!-- BNO055 IMU sensor macro -->
-  <xacro:macro name="bno055_v0" params="name parent *origin">
+  <xacro:macro name="bno055_imu_v0" params="name parent *origin">
     <!-- ZED -->
     <joint name="${name}_joint" type="fixed">
