Commit message: Added LIDAR xacro macros to car URDF files #23

File: gigatron_hardware/urdf/gigatron.urdf.xacro (robot description, xacro)
@@ -7,4 +7,5 @@
     <xacro:include filename="$(find gigatron_hardware)/urdf/sensors/bno055_imu.urdf.xacro" />
     <xacro:include filename="$(find gigatron_hardware)/urdf/sensors/rplidar.urdf.xacro" />
+    <xacro:include filename="$(find gigatron_hardware)/urdf/sensors/xvlidar.urdf.xacro" />
     <!-- Note: Base Link is the center of the robot, right under the batteries. -->
     <!-- Physical Constant Macros -->
@@ -24,14 +25,20 @@
     <xacro:property name="imu_y" value="0" />
     <xacro:property name="imu_z" value="-0.0254" />
-    <!-- LIDAR placement relative to base_link -->
-    <xacro:property name="lidar_x" value=".5588" />
-    <xacro:property name="lidar_y" value="0" />
-    <xacro:property name="lidar_z" value="0.2286" />
-    <xacro:property name="lidar_yaw" value="0" />
-    <!-- Rear LIDAR placement relative to base_link -->
-    <xacro:property name="back_lidar_x" value="-0.5334" />
-    <xacro:property name="back_lidar_y" value="0" />
-    <xacro:property name="back_lidar_z" value="0.3048" />
-    <xacro:property name="back_lidar_yaw" value="0" />
+    <!-- XV LIDAR low-mounted on front, placement relative to base_link -->
+    <xacro:property name="xvlidar_x" value="-0.5334" /> <!-- TODO: actual values -->
+    <xacro:property name="xvlidar_y" value="0" />
+    <xacro:property name="xvlidar_z" value="0.3048" />
+    <xacro:property name="xvlidar_roll" value="0" />
+    <xacro:property name="xvlidar_pitch" value="0" />
+    <xacro:property name="xvlidar_yaw" value="0" />
+    <!--RPLIDAR placement relative to base_link --> <!-- TODO: are we even using this? -->
+<!--
+    <xacro:property name="rplidar_x" value=".5588" />
+    <xacro:property name="rplidar_y" value="0" />
+    <xacro:property name="rplidar_z" value="0.2286" />
+    <xacro:property name="rplidar_roll" value="0" />
+    <xacro:property name="rplidar_pitch" value="0" />
+    <xacro:property name="rplidar_yaw" value="0" />
+-->
     <!-- ZED placement relative to base_link -->
     <xacro:property name="zed_x" value="-0.0254" />
@@ -123,11 +130,11 @@
     </link>
     <!-- the back left wheel -->
-    <joint name="back_left_wheel_joint" type="fixed" >
+    <joint name="low_left_wheel_joint" type="fixed" >
         <!-- <axis xyz="0 1 0" /> -->
         <parent link="base_link" />
-        <child link="back_left_wheel_link" />
+        <child link="low_left_wheel_link" />
         <origin xyz="-${wheelbase_length/2} ${wheelbase_width/2} -${wheel_radius}" rpy="0 0 0" /> <!-- ? -->
     </joint>
-    <link name="back_left_wheel_link">
+    <link name="low_left_wheel_link">
         <inertial>
             <mass value="0.01" />
@@ -150,89 +157,61 @@
     </link>
     <!-- the back right wheel -->
-    <joint name="back_right_wheel_joint" type="fixed" >
+    <joint name="low_right_wheel_joint" type="fixed" >
         <!-- <axis xyz="0 1 0" /> -->
         <parent link="base_link" />
-        <child link="back_right_wheel_link" />
+        <child link="low_right_wheel_link" />
         <origin xyz="-${wheelbase_length/2} -${wheelbase_width/2} -${wheel_radius}" rpy="0 0 0" /> <!-- ? -->
     </joint>
-    <link name="back_right_wheel_link">
-        <inertial>
-            <mass value="0.01" />
-            <origin xyz="0 0 0" />
-            <inertia  ixx="0.01" ixy="0.0"  ixz="0.0"  iyy="0.01"  iyz="0.0"  izz="0.01" />
-        </inertial>
-        <visual>
-            <origin xyz="0 0 0" rpy="${M_PI/2} 0 0" />
-            <geometry>
-                <cylinder radius="${wheel_radius}" length="${wheel_width}" />
-            </geometry>
-            <material name="Black"/>
-        </visual>
-        <collision>
-            <origin xyz="0 0 0" rpy="${M_PI/2} 0 0" />
-            <geometry>
-                <cylinder radius="${wheel_radius}" length="${wheel_width}" />
-            </geometry>
-        </collision>
-    </link>
-    <!-- LIDAR -->
-    <joint name="laser_base_mount_joint" type="fixed">
-        <origin xyz="${lidar_x} ${lidar_y} ${lidar_z}" rpy="0 0 ${lidar_yaw}" />
-        <parent link="base_link"/>
-        <child link="laser_link"/>
-    </joint>
-    <link name="laser_link" type="fixed">
-        <inertial>
-            <mass value="0.1"/>
-            <origin xyz="0 0 0.0"/>
-            <inertia ixx="0.1" ixy="0" ixz="0" iyy="0.1" iyz="0" izz="0.1"/>
-        </inertial>
-        <visual>
-            <origin rpy="0 0 0" xyz="0 0 0.02"/>
-            <geometry>
-                <cylinder radius="0.04" length="0.03175"/>
-            </geometry>
-            <material name="DarkGrey"/>
-        </visual>
-        <collision>
-            <origin rpy="0 0 0" xyz="0 0 0.025"/>
-            <geometry>
-                <box size="0.05 0.05 0.05"/>
-            </geometry>
-        </collision>
-    </link>
-    <!-- BACK LIDAR -->
-    <joint name="back_laser_base_mount_joint" type="fixed">
-        <origin xyz="${back_lidar_x} ${back_lidar_y} ${back_lidar_z}" rpy="0 0 ${back_lidar_yaw}" />
-        <parent link="base_link"/>
-        <child link="back_laser_link"/>
-    </joint>
-    <link name="back_laser_link" type="fixed">
-        <inertial>
-            <mass value="0.1"/>
-            <origin xyz="0 0 0.0"/>
-            <inertia ixx="0.1" ixy="0" ixz="0" iyy="0.1" iyz="0" izz="0.1"/>
-        </inertial>
-        <visual>
-            <origin rpy="0 0 0" xyz="0 0 0.02"/>
-            <geometry>
-                <cylinder radius="0.04" length="0.03175"/>
-            </geometry>
-            <material name="DarkGrey"/>
-        </visual>
-        <collision>
-            <origin rpy="0 0 0" xyz="0 0 0.025"/>
-            <geometry>
-                <box size="0.05 0.05 0.05"/>
-            </geometry>
-        </collision>
-    </link>
+    <link name="low_right_wheel_link">
+        <inertial>
+            <mass value="0.01" />
+            <origin xyz="0 0 0" />
+            <inertia  ixx="0.01" ixy="0.0"  ixz="0.0"  iyy="0.01"  iyz="0.0"  izz="0.01" />
+        </inertial>
+        <visual>
+            <origin xyz="0 0 0" rpy="${M_PI/2} 0 0" />
+            <geometry>
+                <cylinder radius="${wheel_radius}" length="${wheel_width}" />
+            </geometry>
+            <material name="Black"/>
+        </visual>
+        <collision>
+            <origin xyz="0 0 0" rpy="${M_PI/2} 0 0" />
+            <geometry>
+                <cylinder radius="${wheel_radius}" length="${wheel_width}" />
+            </geometry>
+        </collision>
+    </link>
+    <!-- RPLIDAR -->
+<!--     <xacro:rplidar_v0
+        name="rplidar"
+        parent="base_link">
+        <origin
+            xyz="${rplidar_x} ${rplidar_y} ${rplidar_z}"
+            rpy="${rplidar_roll} ${rplidar_pitch} ${rplidar_yaw}" />
+    </xacro:rplidar_v0> -->
+    <!-- XV LIDAR -->
+    <xacro:xvlidar_v0
+        name="xvlidar"
+        parent="base_link">
+        <origin
+            xyz="${xvlidar_x} ${xvlidar_y} ${xvlidar_z}"
+            rpy="${xvlidar_roll} ${xvlidar_pitch} ${xvlidar_yaw}" />
+    </xacro:xvlidar_v0>
     <!-- IMU -->
-    <xacro:bno055_imu_v0 name="imu" parent="base_link">
-        <origin xyz="${imu_x} ${imu_y} ${imu_z}" rpy="0 0 0" />
+    <xacro:bno055_imu_v0
+        name="imu"
+        parent="base_link">
+        <origin
+            xyz="${imu_x} ${imu_y} ${imu_z}"
+            rpy="0 0 0" />
     </xacro:bno055_imu_v0>
     <!-- ZED -->
-    <xacro:zed_v0 name="zed" parent="base_link">
-        <origin xyz="${zed_x} ${zed_y} ${zed_z}" rpy="0 0 0" />
+    <xacro:zed_v0
+        name="zed"
+        parent="base_link">
+        <origin
+            xyz="${zed_x} ${zed_y} ${zed_z}"
+            rpy="0 0 0" />
     </xacro:zed_v0>
 </robot>

File: gigatron_hardware/urdf/kilotron.urdf.xacro (robot description, xacro)
@@ -165,37 +165,27 @@
         </collision>
     </link>
-    <!-- LIDAR -->
-    <joint name="laser_base_mount_joint" type="fixed">
-        <origin xyz="${lidar_x} ${lidar_y} ${lidar_z}" rpy="0 0 ${lidar_yaw}" />
-        <parent link="base_link"/>
-        <child link="laser_link"/>
-    </joint>
-    <link name="laser_link" type="fixed">
-        <inertial>
-            <mass value="0.1"/>
-            <origin xyz="0 0 0.0"/>
-            <inertia ixx="0.1" ixy="0" ixz="0" iyy="0.1" iyz="0" izz="0.1"/>
-        </inertial>
-        <visual>
-            <origin rpy="0 0 0" xyz="0 0 0.02"/>
-            <geometry>
-                <cylinder radius="0.04" length="0.03175"/>
-            </geometry>
-            <material name="DarkGrey"/>
-        </visual>
-        <collision>
-            <origin rpy="0 0 0" xyz="0 0 0.025"/>
-            <geometry>
-                <box size="0.05 0.05 0.05"/>
-            </geometry>
-        </collision>
-    </link>
+    <!-- XV LIDAR -->
+    <xacro:rplidar_v0
+        name="rplidar"
+        parent="base_link">
+        <origin
+            xyz="${lidar_x} ${lidar_y} ${lidar_z}"
+            rpy="0 0 ${lidar_yaw}" />
+    </xacro:rplidar_v0>
     <!-- IMU -->
-    <xacro:bno055_imu_v0 name="imu" parent="base_link">
-        <origin xyz="${imu_x} ${imu_y} ${imu_z}" rpy="0 0 0" />
+    <xacro:bno055_imu_v0
+        name="imu"
+        parent="base_link">
+        <origin
+            xyz="${imu_x} ${imu_y} ${imu_z}"
+            rpy="0 0 0" />
     </xacro:bno055_imu_v0>
     <!-- ZED -->
-    <xacro:zed_v0 name="zed" parent="base_link">
-        <origin xyz="${zed_x} ${zed_y} ${zed_z}" rpy="0 0 0" />
+    <xacro:zed_v0
+        name="zed"
+        parent="base_link">
+        <origin
+            xyz="${zed_x} ${zed_y} ${zed_z}"
+            rpy="0 0 0" />
     </xacro:zed_v0>
 </robot>

Commit message: Added proper location for XV LIDAR and ZED on Gigatron #23

File: gigatron_hardware/urdf/gigatron.urdf.xacro (robot description, xacro)
@@ -21,13 +21,13 @@
     <xacro:property name="wheel_radius" value="0.12446" /> <!-- 4.9" -->
     <xacro:property name="wheel_width" value="0.075" />
-    <!-- IMU placement relative to base_link -->
+    <!-- IMU placement relative to base_link --> <!-- TODO: actual values -->
     <xacro:property name="imu_x" value="0" />
     <xacro:property name="imu_y" value="0" />
     <xacro:property name="imu_z" value="-0.0254" />
     <!-- XV LIDAR low-mounted on front, placement relative to base_link -->
-    <xacro:property name="xvlidar_x" value="-0.5334" /> <!-- TODO: actual values -->
+    <xacro:property name="xvlidar_x" value="${wheelbase_length/2 + 0.19}" />
     <xacro:property name="xvlidar_y" value="0" />
-    <xacro:property name="xvlidar_z" value="0.3048" />
-    <xacro:property name="xvlidar_roll" value="0" />
+    <xacro:property name="xvlidar_z" value="-0.3" />
+    <xacro:property name="xvlidar_roll" value="${M_PI/2}" />
     <xacro:property name="xvlidar_pitch" value="0" />
     <xacro:property name="xvlidar_yaw" value="0" />
@@ -42,7 +42,7 @@
 -->
     <!-- ZED placement relative to base_link -->
-    <xacro:property name="zed_x" value="-0.0254" />
+    <xacro:property name="zed_x" value="0.19" />
     <xacro:property name="zed_y" value="0.0" />
-    <xacro:property name="zed_z" value="0.27942" />
+    <xacro:property name="zed_z" value="0.36" />
     <!-- Main body -->
     <link name="base_link">

File: gigatron_hardware/urdf/kilotron.urdf.xacro (robot description, xacro)
@@ -165,5 +165,5 @@
         </collision>
     </link>
-    <!-- XV LIDAR -->
+    <!-- RPLIDAR -->
     <xacro:rplidar_v0
         name="rplidar"

Commit message: Updates in gigatron launch file and fix in URDF LIDAR roll #23

File: gigatron_hardware/urdf/gigatron.urdf.xacro (robot description, xacro)
@@ -29,5 +29,5 @@
     <xacro:property name="xvlidar_y" value="0" />
     <xacro:property name="xvlidar_z" value="-0.3" />
-    <xacro:property name="xvlidar_roll" value="${M_PI/2}" />
+    <xacro:property name="xvlidar_roll" value="${M_PI}" />
     <xacro:property name="xvlidar_pitch" value="0" />
     <xacro:property name="xvlidar_yaw" value="0" />

Commit message: Updated XV LUDAR yaw on Gigatron #23

File: gigatron_hardware/urdf/gigatron.urdf.xacro (robot description, xacro)
@@ -31,5 +31,5 @@
     <xacro:property name="xvlidar_roll" value="${M_PI}" />
     <xacro:property name="xvlidar_pitch" value="0" />
-    <xacro:property name="xvlidar_yaw" value="0" />
+    <xacro:property name="xvlidar_yaw" value="${M_PI}" />
     <!--RPLIDAR placement relative to base_link --> <!-- TODO: are we even using this? -->
 <!--

Commit message: renabled rplidar in urdf

File: gigatron_hardware/urdf/gigatron.urdf.xacro (robot description, xacro)
@@ -33,5 +33,4 @@
     <xacro:property name="xvlidar_yaw" value="${M_PI}" />
     <!--RPLIDAR placement relative to base_link --> <!-- TODO: are we even using this? -->
-<!--
     <xacro:property name="rplidar_x" value=".5588" />
     <xacro:property name="rplidar_y" value="0" />
@@ -39,6 +38,5 @@
     <xacro:property name="rplidar_roll" value="0" />
     <xacro:property name="rplidar_pitch" value="0" />
-    <xacro:property name="rplidar_yaw" value="0" />
--->
+    <xacro:property name="rplidar_yaw" value="0" /> <!-- ${M_PI} -->
     <!-- ZED placement relative to base_link -->
     <xacro:property name="zed_x" value="0.19" />
@@ -184,5 +182,5 @@
     </link>
     <!-- RPLIDAR -->
-<!--     <xacro:rplidar_v0
+    <xacro:rplidar_v0
         name="rplidar"
         parent="base_link">
@@ -190,5 +188,5 @@
             xyz="${rplidar_x} ${rplidar_y} ${rplidar_z}"
             rpy="${rplidar_roll} ${rplidar_pitch} ${rplidar_yaw}" />
-    </xacro:rplidar_v0> -->
+    </xacro:rplidar_v0>
     <!-- XV LIDAR -->
     <xacro:xvlidar_v0

Commit message: Updated IMU placement in URDF

File: gigatron_hardware/urdf/gigatron.urdf.xacro (robot description, xacro)
@@ -21,8 +21,8 @@
     <xacro:property name="wheel_radius" value="0.12446" /> <!-- 4.9" -->
     <xacro:property name="wheel_width" value="0.075" />
-    <!-- IMU placement relative to base_link --> <!-- TODO: actual values -->
-    <xacro:property name="imu_x" value="0" />
-    <xacro:property name="imu_y" value="0" />
-    <xacro:property name="imu_z" value="-0.0254" />
+    <!-- IMU placement relative to base_link -->
+    <xacro:property name="imu_x" value="${-wheelbase_length/2 - 0.19}" />
+    <xacro:property name="imu_y" value="-0.035" />
+    <xacro:property name="imu_z" value="0.3" />
     <!-- XV LIDAR low-mounted on front, placement relative to base_link -->
     <xacro:property name="xvlidar_x" value="${wheelbase_length/2 + 0.19}" />
@@ -32,5 +32,5 @@
     <xacro:property name="xvlidar_pitch" value="0" />
     <xacro:property name="xvlidar_yaw" value="${M_PI}" />
-    <!--RPLIDAR placement relative to base_link --> <!-- TODO: are we even using this? -->
+    <!--RPLIDAR placement relative to base_link -->
     <xacro:property name="rplidar_x" value=".5588" />
     <xacro:property name="rplidar_y" value="0" />
@@ -38,5 +38,5 @@
     <xacro:property name="rplidar_roll" value="0" />
     <xacro:property name="rplidar_pitch" value="0" />
-    <xacro:property name="rplidar_yaw" value="0" /> <!-- ${M_PI} -->
+    <xacro:property name="rplidar_yaw" value="0" />
     <!-- ZED placement relative to base_link -->
     <xacro:property name="zed_x" value="0.19" />

Commit message: Fixed gigatron URDF XV LIDAR location

File: gigatron_hardware/urdf/gigatron.urdf.xacro (robot description, xacro)
@@ -28,5 +28,5 @@
     <xacro:property name="xvlidar_x" value="${wheelbase_length/2 + 0.19}" />
     <xacro:property name="xvlidar_y" value="0" />
-    <xacro:property name="xvlidar_z" value="-0.3" />
+    <xacro:property name="xvlidar_z" value="-0.03" />
     <xacro:property name="xvlidar_roll" value="${M_PI}" />
     <xacro:property name="xvlidar_pitch" value="0" />
@@ -51,8 +51,8 @@
         </inertial>
         <visual>
-            <origin xyz="0 0 0" rpy="0 0 0" />
-            <geometry>
-                <box size="${car_length} ${wheelbase_width} ${car_height}" />
-            </geometry>
+            <origin xyz="0 0 ${car_height/4+0.02}" rpy="0 0 0" />
+            <geometry>
+                 <box size="${car_length} ${wheelbase_width} ${car_height}" />
+             </geometry>
             <material name="Grey"/>
         </visual>

Commit message: Updated URDF for remounted RPLIDAR #25

File: gigatron_hardware/urdf/gigatron.urdf.xacro (robot description, xacro)
@@ -25,13 +25,13 @@
     <xacro:property name="imu_y" value="-0.035" />
     <xacro:property name="imu_z" value="0.3" />
-    <!-- XV LIDAR low-mounted on front, placement relative to base_link -->
-    <xacro:property name="xvlidar_x" value="${wheelbase_length/2 + 0.19}" />
-    <xacro:property name="xvlidar_y" value="0" />
-    <xacro:property name="xvlidar_z" value="-0.03" />
-    <xacro:property name="xvlidar_roll" value="${M_PI}" />
-    <xacro:property name="xvlidar_pitch" value="0" />
-    <xacro:property name="xvlidar_yaw" value="${M_PI}" />
+    <!-- RPLIDAR low-mounted on front, placement relative to base_link -->
+    <xacro:property name="rplidar_x" value="${wheelbase_length/2 + 0.19}" />
+    <xacro:property name="rplidar_y" value="0" />
+    <xacro:property name="rplidar_z" value="-0.03" />
+    <xacro:property name="rplidar_roll" value="${M_PI}" />
+    <xacro:property name="rplidar_pitch" value="0" />
+    <xacro:property name="rplidar_yaw" value="${M_PI}" />
     <!--RPLIDAR placement relative to base_link -->
-    <xacro:property name="rplidar_x" value=".5588" />
+<!--     <xacro:property name="rplidar_x" value=".5588" />
     <xacro:property name="rplidar_y" value="0" />
     <xacro:property name="rplidar_z" value="0.2286" />
@@ -39,5 +39,6 @@
     <xacro:property name="rplidar_pitch" value="0" />
     <xacro:property name="rplidar_yaw" value="0" />
-    <!-- ZED placement relative to base_link -->
+-->
+     <!-- ZED placement relative to base_link -->
     <xacro:property name="zed_x" value="0.19" />
     <xacro:property name="zed_y" value="0.0" />
@@ -190,5 +191,5 @@
     </xacro:rplidar_v0>
     <!-- XV LIDAR -->
-    <xacro:xvlidar_v0
+<!--     <xacro:xvlidar_v0
         name="xvlidar"
         parent="base_link">
@@ -196,5 +197,5 @@
             xyz="${xvlidar_x} ${xvlidar_y} ${xvlidar_z}"
             rpy="${xvlidar_roll} ${xvlidar_pitch} ${xvlidar_yaw}" />
-    </xacro:xvlidar_v0>
+    </xacro:xvlidar_v0> -->
     <!-- IMU -->
     <xacro:bno055_imu_v0

Commit message: Removed outdated LIDAR logic from launch file and URDF #28

File: gigatron_hardware/urdf/gigatron.urdf.xacro (robot description, xacro)
@@ -26,10 +26,10 @@
     <xacro:property name="imu_z" value="0.3" />
     <!-- XV LIDAR low-mounted on front, placement relative to base_link -->
-    <xacro:property name="xvlidar_x" value="${wheelbase_length/2 + 0.19}" />
+<!--     <xacro:property name="xvlidar_x" value="${wheelbase_length/2 + 0.19}" />
     <xacro:property name="xvlidar_y" value="0" />
     <xacro:property name="xvlidar_z" value="-0.03" />
     <xacro:property name="xvlidar_roll" value="${M_PI}" />
     <xacro:property name="xvlidar_pitch" value="0" />
-    <xacro:property name="xvlidar_yaw" value="${M_PI}" />
+    <xacro:property name="xvlidar_yaw" value="${M_PI}" /> -->
     <!--RPLIDAR placement relative to base_link -->
     <xacro:property name="rplidar_x" value=".5588" />
