Commit message: Centered and rotated RPLIDAR mesh and added to URDF

File: gigatron_hardware/urdf/sensors/rplidar.urdf.xacro (robot description, xacro)
@@ -18,5 +18,6 @@
             <origin rpy="0 0 0" xyz="0 0 0.02"/>
             <geometry>
-                <cylinder radius="0.035" length="0.035"/>
+                <!-- <cylinder radius="0.035" length="0.035"/> -->
+                <mesh filename="package://gigatron_hardware/meshes/rplidar.stl" />
             </geometry>
             <material name="DarkGrey"/>
